File: runar.kicad_sch (KiCad schematic)
At the start: 44 parts, among them SW1 SW_Push_45deg, SW10 SW_Push_45deg, SW11 SW_Push_45deg, SW12 SW_Push_45deg, SW13 SW_Push_45deg, SW14 SW_Push_45deg, SW15 SW_Push_45deg, SW16 SW_Push_45deg, SW17 SW_Push_45deg, SW18 MLL1200S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

Commit message: few final touches to silkscreen
Other:
- moved on the sheet: JP16, JP20
Changed lines of the file:
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@@
 	(wire
 		(pts
-			(xy 187.96 124.46) (xy 187.96 128.27)
-		)
-		(stroke
-			(width 0)
-			(type default)
-		)
-	)
-	(wire
-		(pts
-			(xy 218.44 107.95) (xy 215.9 107.95)
-		)
-		(stroke
-			(width 0)
-			(type default)
-		)
-	)
-	(wire
-		(pts
 			(xy 218.44 73.66) (xy 215.9 73.66)
 		)
@@
 	(wire
 		(pts
-			(xy 215.9 124.46) (xy 215.9 128.27)
-		)
-		(stroke
-			(width 0)
-			(type default)
-		)
-	)
-	(wire
-		(pts
 			(xy 163.83 74.93) (xy 166.37 74.93)
 		)
@@
 	(wire
 		(pts
-			(xy 190.5 107.95) (xy 187.96 107.95)
-		)
-		(stroke
-			(width 0)
-			(type default)
-		)
-	)
-	(wire
-		(pts
 			(xy 210.82 39.37) (xy 204.47 39.37)
 		)
@@
 	(wire
 		(pts
-			(xy 185.42 128.27) (xy 187.96 128.27)
+			(xy 185.42 110.49) (xy 187.96 110.49)
 		)
 		(stroke
@@
 	(wire
 		(pts
-			(xy 190.5 124.46) (xy 187.96 124.46)
-		)
-		(stroke
-			(width 0)
-			(type default)
-		)
-	)
-	(wire
-		(pts
-			(xy 213.36 128.27) (xy 215.9 128.27)
-		)
-		(stroke
-			(width 0)
-			(type default)
-		)
-	)
-	(wire
-		(pts
-			(xy 215.9 104.14) (xy 215.9 107.95)
-		)
-		(stroke
-			(width 0)
-			(type default)
-		)
-	)
-	(wire
-		(pts
-			(xy 218.44 124.46) (xy 215.9 124.46)
-		)
-		(stroke
-			(width 0)
-			(type default)
-		)
-	)
-	(wire
-		(pts
-			(xy 187.96 104.14) (xy 187.96 107.95)
+			(xy 213.36 110.49) (xy 215.9 110.49)
 		)
 		(stroke
@@
 	(global_label "SW10"
 		(shape input)
-		(at 205.74 128.27 180)
+		(at 205.74 110.49 180)
 		(fields_autoplaced yes)
 		(effects
@@
 		)
 		(property "Intersheetrefs" "${INTERSHEET_REFS}"
-			(at 197.6749 128.27 0)
+			(at 197.6749 110.49 0)
 			(effects
 				(font
@@
 	(global_label "21"
 		(shape input)
-		(at 190.5 124.46 0)
+		(at 187.96 110.49 0)
 		(fields_autoplaced yes)
 		(effects
@@
 		)
 		(property "Intersheetrefs" "${INTERSHEET_REFS}"
-			(at 195.9042 124.46 0)
+			(at 193.3642 110.49 0)
 			(effects
 				(font
@@
 	(global_label "5"
 		(shape input)
-		(at 218.44 107.95 0)
+		(at 215.9 104.14 0)
 		(fields_autoplaced yes)
 		(effects
@@
 		)
 		(property "Intersheetrefs" "${INTERSHEET_REFS}"
-			(at 222.6347 107.95 0)
+			(at 220.0947 104.14 0)
 			(effects
 				(font
@@
 	(global_label "4"
 		(shape input)
-		(at 190.5 107.95 0)
+		(at 187.96 104.14 0)
 		(fields_autoplaced yes)
 		(effects
@@
 		)
 		(property "Intersheetrefs" "${INTERSHEET_REFS}"
-			(at 194.6947 107.95 0)
+			(at 192.1547 104.14 0)
 			(effects
 				(font
@@
 	(global_label "20"
 		(shape input)
-		(at 218.44 124.46 0)
+		(at 215.9 110.49 0)
 		(fields_autoplaced yes)
 		(effects
@@
 		)
 		(property "Intersheetrefs" "${INTERSHEET_REFS}"
-			(at 223.8442 124.46 0)
+			(at 221.3042 110.49 0)
 			(effects
 				(font
@@
 	(symbol
 		(lib_id "Jumper:SolderJumper_2_Open")
-		(at 209.55 128.27 0)
+		(at 209.55 110.49 0)
 		(unit 1)
 		(exclude_from_sim no)
@@
 		(dnp no)
 		(property "Reference" "JP20"
-			(at 209.55 125.984 0)
+			(at 209.55 108.204 0)
 			(effects
 				(font
@@
 		)
 		(property "Value" "SolderJumper_2_Open"
-			(at 209.55 124.46 0)
+			(at 209.55 106.68 0)
 			(effects
 				(font
@@
 		)
 		(property "Footprint" "BLE_KBD:Solder_Jumper"
-			(at 209.55 128.27 0)
+			(at 209.55 110.49 0)
 			(effects
 				(font
@@
 		)
 		(property "Datasheet" "~"
-			(at 209.55 128.27 0)
+			(at 209.55 110.49 0)
 			(effects
 				(font
@@
 		)
 		(property "Description" "Solder Jumper, 2-pole, open"
-			(at 209.55 128.27 0)
+			(at 209.55 110.49 0)
 			(effects
 				(font
@@
 	(symbol
 		(lib_id "Jumper:SolderJumper_2_Open")
-		(at 181.61 128.27 0)
+		(at 181.61 110.49 0)
 		(unit 1)
 		(exclude_from_sim no)
@@
 		(dnp no)
 		(property "Reference" "JP16"
-			(at 181.61 125.984 0)
+			(at 181.61 108.204 0)
 			(effects
 				(font
@@
 		)
 		(property "Value" "SolderJumper_2_Open"
-			(at 181.61 124.46 0)
+			(at 181.61 106.68 0)
 			(effects
 				(font
@@
 		)
 		(property "Footprint" "BLE_KBD:Solder_Jumper"
-			(at 181.61 128.27 0)
+			(at 181.61 110.49 0)
 			(effects
 				(font
@@
 		)
 		(property "Datasheet" "~"
-			(at 181.61 128.27 0)
+			(at 181.61 110.49 0)
 			(effects
 				(font
@@
 		)
 		(property "Description" "Solder Jumper, 2-pole, open"
-			(at 181.61 128.27 0)
+			(at 181.61 110.49 0)
 			(effects
 				(font
@@
 	(symbol
 		(lib_id "power:GND")
-		(at 177.8 128.27 270)
+		(at 177.8 110.49 270)
 		(unit 1)
 		(exclude_from_sim no)
@@
 		(dnp no)
 		(property "Reference" "#PWR030"
-			(at 171.45 128.27 0)
+			(at 171.45 110.49 0)
 			(effects
 				(font
@@
 		)
 		(property "Value" "GND"
-			(at 173.99 128.27 0)
+			(at 173.99 110.49 0)
 			(effects
 				(font
@@
 		)
 		(property "Footprint" ""
-			(at 177.8 128.27 0)
+			(at 177.8 110.49 0)
 			(effects
 				(font
@@
 		)
 		(property "Datasheet" ""
-			(at 177.8 128.27 0)
+			(at 177.8 110.49 0)
 			(effects
 				(font
@@
 		)
 		(property "Description" "Power symbol creates a global label with name \"GND\" , ground"
-			(at 177.8 128.27 0)
+			(at 177.8 110.49 0)
 			(effects
 				(font
